Commit message: 105

File: description/robot_core.xacro (robot description, xacro)
@@ -73,5 +73,5 @@
         <parent link="base_link"/>
         <child link="left_wheel_2"/>
-        <origin xyz="0.109 ${wheel_offset_y} 0" rpy="-${pi/2} 0 0" />
+        <origin xyz="0.105 ${wheel_offset_y} 0" rpy="-${pi/2} 0 0" />
         <axis xyz="0 0 1"/>
     </joint>
@@ -151,5 +151,5 @@
         <parent link="base_link"/>
         <child link="right_wheel"/>
-        <origin xyz="0.109 ${-wheel_offset_y} 0" rpy="${pi/2} 0 0" />
+        <origin xyz="0.105 ${-wheel_offset_y} 0" rpy="${pi/2} 0 0" />
         <axis xyz="0 0 -1"/>
     </joint>

Commit message: Bimo

File: description/robot_core.xacro (robot description, xacro)
@@ -9,11 +9,11 @@
     <xacro:property name="wheel_thickness" value="0.045"/>
     <xacro:property name="wheel_mass" value="0.01"/>
-    <xacro:property name="wheel_offset_x" value="0.030"/>
-    <xacro:property name="wheel_offset_y" value="0.065"/>
+    <xacro:property name="wheel_offset_x" value="0.0525"/>
+    <xacro:property name="wheel_offset_y" value="0.06"/>
     <xacro:property name="wheel_offset_z" value="0.01"/>
     <xacro:property name="caster_wheel_radius" value="0.01"/>
-    <xacro:property name="caster_wheel_mass" value="0.01"/>
+    <!--xacro:property name="caster_wheel_mass" value="0.01"/>
     <xacro:property name="caster_wheel_offset_x" value="0.075"/>
-    <xacro:property name="caster_wheel_offset_z" value="${wheel_offset_z - wheel_radius + caster_wheel_radius}"/>
+    <xacro:property name="caster_wheel_offset_z" value="${wheel_offset_z - wheel_radius + caster_wheel_radius}"/-->
     <material name="white">
         <color rgba="1 1 1 1" />
@@ -46,5 +46,5 @@
         <parent link="base_link"/>
         <child link="chassis"/>
-        <origin xyz="${-wheel_offset_x} 0 ${-wheel_offset_z}"/>
+        <origin xyz="${-chassis_length/2} 0 ${-wheel_offset_z}"/>
     </joint>
     <link name="chassis">
@@ -73,5 +73,5 @@
         <parent link="base_link"/>
         <child link="left_wheel_2"/>
-        <origin xyz="0.105 ${wheel_offset_y} 0" rpy="-${pi/2} 0 0" />
+        <origin xyz="${-wheel_offset_x} ${-wheel_offset_y} 0" rpy="-${pi/2} 0 0" />
         <axis xyz="0 0 1"/>
     </joint>
@@ -99,5 +99,5 @@
         <parent link="base_link"/>
         <child link="left_wheel"/>
-        <origin xyz="0 ${wheel_offset_y} 0" rpy="-${pi/2} 0 0" />
+        <origin xyz="${wheel_offset_x} ${-wheel_offset_y} 0" rpy="-${pi/2} 0 0" />
         <axis xyz="0 0 1"/>
     </joint>
@@ -125,5 +125,5 @@
         <parent link="base_link"/>
         <child link="right_wheel_2"/>
-        <origin xyz="0 ${-wheel_offset_y} 0" rpy="${pi/2} 0 0" />
+        <origin xyz="${wheel_offset_x} ${wheel_offset_y} 0" rpy="${pi/2} 0 0" />
         <axis xyz="0 0 -1"/>
     </joint>
@@ -151,5 +151,5 @@
         <parent link="base_link"/>
         <child link="right_wheel"/>
-        <origin xyz="0.105 ${-wheel_offset_y} 0" rpy="${pi/2} 0 0" />
+        <origin xyz="${-wheel_offset_x} ${wheel_offset_y} 0" rpy="${pi/2} 0 0" />
         <axis xyz="0 0 -1"/>
     </joint>

File: description/ros2_control.xacro (robot description, xacro)
@@ -11,5 +11,5 @@
                 <param name="baud_rate">57600</param>
                 <param name="timeout">1000</param>
-                <param name="enc_counts_per_rev">1977</param>
+                <param name="enc_counts_per_rev">3954</param>
             </hardware>
             <joint name="left_wheel_joint">

Commit message: modify

File: description/robot_core.xacro (robot description, xacro)
@@ -10,5 +10,5 @@
     <xacro:property name="wheel_mass" value="0.01"/>
     <xacro:property name="wheel_offset_x" value="0.0525"/>
-    <xacro:property name="wheel_offset_y" value="0.06"/>
+    <xacro:property name="wheel_offset_y" value="0.065"/>
     <xacro:property name="wheel_offset_z" value="0.01"/>
     <xacro:property name="caster_wheel_radius" value="0.01"/>

Commit message: joy_stick

File: description/robot_core.xacro (robot description, xacro)
@@ -12,6 +12,6 @@
     <xacro:property name="wheel_offset_y" value="0.065"/>
     <xacro:property name="wheel_offset_z" value="0.01"/>
-    <xacro:property name="caster_wheel_radius" value="0.01"/>
-    <!--xacro:property name="caster_wheel_mass" value="0.01"/>
+    <!--xacro:property name="caster_wheel_radius" value="0.01"/>
+    <xacro:property name="caster_wheel_mass" value="0.01"/>
     <xacro:property name="caster_wheel_offset_x" value="0.075"/>
     <xacro:property name="caster_wheel_offset_z" value="${wheel_offset_z - wheel_radius + caster_wheel_radius}"/-->
