Commit message: robot_core

File: description/gazebo_control.xacro (robot description, xacro)
@@ -6,5 +6,5 @@
             <left_joint>left_wheel_joint</left_joint>
             <right_joint>right_wheel_joint</right_joint>
-            <wheel_separation>0.085</wheel_separation>
+            <wheel_separation>0.092</wheel_separation>
             <wheel_diameter>0.060</wheel_diameter>
             <!-- Limits -->

File: description/robot_core.xacro (robot description, xacro)
@@ -3,12 +3,12 @@
     <xacro:include filename="inertial_macros.xacro"/>
     <xacro:property name="chassis_length" value="0.165"/>
-    <xacro:property name="chassis_width" value="0.085"/>
+    <xacro:property name="chassis_width" value="0.092"/>
     <xacro:property name="chassis_height" value="0.080"/>
-    <xacro:property name="chassis_mass" value="1.0"/>
+    <xacro:property name="chassis_mass" value="2.0"/>
     <xacro:property name="wheel_radius" value="0.030"/>
     <xacro:property name="wheel_thickness" value="0.045"/>
-    <xacro:property name="wheel_mass" value="0.01"/>
+    <xacro:property name="wheel_mass" value="0.1"/>
     <xacro:property name="wheel_offset_x" value="0.0525"/>
-    <xacro:property name="wheel_offset_y" value="0.065"/>
+    <xacro:property name="wheel_offset_y" value="0.0685"/>
     <xacro:property name="wheel_offset_z" value="0.01"/>
     <!--xacro:property name="caster_wheel_radius" value="0.01"/>
